File: modulovier.kicad_sch (KiCad schematic)
At the start: 19 parts, among them J1 EXT. PORT, J2 oled, J3 leds, SW1 mx, SW2 mx, SW3 mx, SW4 mx, SW5 volume, U2 Pico

Commit message: update schema
Parts:
- added U?: WeAct-RP2040-Pico, WeAct-RP2040-Pico:WeAct-RP2040-Pico, symbol RP2040:WeAct-RP2040-Pico
Connections:
- net 5V: now also U?.40 (VBUS)
- net SCL: now also U?.21 (GP16)
- net SDA: now also U?.22 (GP17)
- net c1: now also U?.27 (GP21)
- net c2: now also U?.29 (GP22)
- net c3: now also U?.31 (GP27)
- net ea: now also U?.25 (GP19)
- net eb: now also U?.24 (GP18)
- net led1: now also U?.12 (GP9)
- net led2: now also U?.11 (GP8)
- net leds_data: now also U?.14 (GP10)
- net r1: now also U?.9 (GP6)
- net r2: now also U?.7 (GP5)
- new net 3.3V: U?.37 (3V3)
Other:
- moved on the sheet: SW5

Commit message: Finished work to verify
Parts:
- removed D5: D, m65:diode_v, symbol Device:D
- removed J1: EXT. PORT, IDC-Header_2x20_P2.54mm_Vertical, symbol Connector_Generic:Conn_02x20_Odd_Even
- removed SW4: mx, m-lego:CherryMX_ChocV2_1u, symbol Switch:SW_Push
- removed U2: Pico, m-lego:RPi_Pico_SMD_TH, symbol m-lego mcus:Pico
- added BZ1: Buzzer, Buzzer_Beeper:Buzzer_12x9.5RM7.6, symbol Device:Buzzer
- D1, D2, D3, D4: footprint m65:diode_v -> Diode_SMD:D_1206_3216Metric_Pad1.42x1.75mm_HandSolder
- D30: footprint m65:LED_D3.0mm_lwr -> M65Lego:LED_D3.0mm_lwr
- D31: footprint m65:LED_D3.0mm_rse -> M65Lego:LED_D3.0mm_rse
- H1: footprint m-lego:LegoHole_12x12u_4875 -> M65Lego:LegoHole_12x12u_4875
- J2: footprint m-lego:OLED_128x32 -> M65Lego:OLED_128x32
- R3, R4: footprint m65:R510_led -> Resistor_SMD:R_1206_3216Metric_Pad1.30x1.75mm_HandSolder
- SW1, SW2, SW3: footprint m65:SW_Cherry_MX_1.00u_PCB-3d -> M65Lego:SW_Cherry_MX_1.00u_PCB
- SW5: footprint m65:RotaryEncoder_Alps_EC11E_Vertical_H20mm -> M65Lego:RotaryEncoder_Alps_EC11E_Vertical_H20mm
- U1: renamed from U?; footprint WeAct-RP2040-Pico:WeAct-RP2040-Pico -> WeAct RP2040:WeAct-RP2040-Pico
Connections:
- net 3.3V is gone; now on net +3V3: U1.37 (3V3)
- net c3 is gone; now on net led2: U1.31 (GP27)
- net gnd is gone; now on net GND: SW5.C
- net GND: now also BZ1.2 (+)
- net SCL: now also U1.20 (GP15); no longer U1.21 (GP16)
- net SDA: now also U1.19 (GP14); no longer U1.22 (GP17)
- net c1: now also U1.25 (GP19); no longer U1.27 (GP21)
- net c2: now also U1.24 (GP18); no longer U1.29 (GP22)
- net ea: now also U1.27 (GP21); no longer U1.25 (GP19)
- net eb: now also U1.26 (GP20); no longer U1.24 (GP18)
- net led1: now also U1.32 (GP28); no longer U1.12 (GP9)
- net led2: no longer U1.11 (GP8)
- net leds_data: now also U1.36 (GP24); no longer U1.14 (GP10)
- net r1: now also U1.29 (GP22); no longer SW5.S2, U1.9 (GP6)
- net r2: now also SW5.S2, U1.22 (GP17); no longer U1.7 (GP5)
- net at D4.1 (K): now also SW5.S1
- net buz: now reaches U1.30 (GP26)
- net buz: now also BZ1.1 (-)
- no-connect marks 2 -> 0
Other:
- note added: "Att : gp28/27 et gnd semblent diff entre pinout schema et empreinte"
- moved on the sheet: SW5, U1
